File: hard/firstVersion/cpuBoard/cpuBoard.sch (KiCad schematic (older format))
At the start: 10 parts

Commit message: Something
Parts:
- removed J?: XLR3_Switched, symbol Connector:XLR3_Switched
- removed U?: 6502, symbol wdc:6502
- added J1: Jumpers, symbol custom:myBus
- added J2: Jumpers, symbol Connector:XLR3_Switched
- added R4: (Not on board), symbol Device:R
- added U1: w65c816s, symbol cpuBoard-rescue:w65c816s-wdc
- D1: renamed from D?; value RED -> GREEN
- gave numbers to parts that had none: 7
Connections:
- net +5V: now also J1.1 (5V), J2.NC, R4.2, U1.3 (ABORT), U1.8 (VDD)
- net GND: now also J1.2 (GND), J2.NO, U1.21 (VSS)
- net VDA: now reaches D2.2 (A)
- net VDA: now also J1.31 (VDA), U1.39 (VDA)
- net IRQ: now reaches R3.2
- net IRQ: now also J1.32 (IRQ), U1.4 (IRQB)
- net RESB: now reaches R5.2, SW1.2
- net RESB: now also J1.29 (RESB), U1.40 (RESB)
- net NMI: now reaches R2.2
- net NMI: now also J1.33 (NMI), U1.6 (NMIB)
- net VPA: now reaches D1.2 (A)
- net VPA: now also J1.30 (VPA), U1.7 (VPA)
- new net: R4.1, U1.2 (RDY)
- new net: J2.N, U1.36 (BE)
- new net A0: J1.18 (A0), U1.9 (A0)
- new net A1: J1.17 (A1), U1.10 (A1)
- new net A10: J1.8 (A10), U1.19 (A10)
- new net A11: J1.7 (A11), U1.20 (A11)
- new net A12: J1.6 (A12), U1.22 (A12)
- new net A13: J1.5 (A13), U1.23 (A13)
- new net A14: J1.4 (A14), U1.24 (A14)
- new net A15: J1.3 (A15), U1.25 (A15)
- new net A2: J1.16 (A2), U1.11 (A2)
- new net A3: J1.15 (A3), U1.12 (A3)
- new net A4: J1.14 (A4), U1.13 (A4)
- new net A5: J1.13 (A5), U1.14 (A5)
- new net A6: J1.12 (A6), U1.15 (A5)
- new net A7: J1.11 (A7), U1.16 (A7)
- new net A8: J1.10 (A8), U1.17 (A8)
- new net A9: J1.9 (A9), U1.18 (A9)
- new net CLK: J1.27 (Clock), U1.37 (PHI2)
- new net D0: J1.26 (D0), U1.33 (D0)
- new net D1: J1.25 (D1), U1.32 (D1)
- new net D2: J1.24 (D2), U1.31 (D2)
- new net D3: J1.23 (D3), U1.30 (D3)
- new net D4: J1.22 (D4), U1.29 (D4)
- new net D5: J1.21 (D5), U1.28 (D5)
- new net D6: J1.20 (D6), U1.27 (D6)
- new net D7: J1.19 (D7), U1.26 (D7)
- new net RWB: J1.28 (RWB), U1.34 (RWB)
Other:
- moved on the sheet: D1, R1
