File: hard/secondVersion/ROM/ROM.sch (KiCad schematic (older format))
At the start: 7 parts, among them J1 XLR3_Switched, J2 myBus, U1 71256SA, U2 4NAND

Commit message: ROM changes
Parts:
- added J3: XLR3_Switched, symbol Connector:XLR3_Switched
Connections:
- net +5V: now also J3.NO
- net GND: now also J3.NC; no longer U1.22 (OEB)
- new net Prog: J3.N, U1.22 (OEB)
- no-connect marks 12 -> 11
Changed lines of the file:
@@
 $EndComp
 $Comp
-L power:GND #PWR05
+L power:GND #PWR07
 U 1 1 60C3EA2F
 P 2350 3100
-F 0 "#PWR05" H 2350 2850 50  0001 C CNN
+F 0 "#PWR07" H 2350 2850 50  0001 C CNN
 F 1 "GND" H 2355 2927 50  0000 C CNN
 F 2 "" H 2350 3100 50  0001 C CNN
@@
 	2350 2850 2350 3000
 $Comp
-L power:+5V #PWR06
+L power:+5V #PWR08
 U 1 1 60C3F0A0
 P 3300 850
-F 0 "#PWR06" H 3300 700 50  0001 C CNN
+F 0 "#PWR08" H 3300 700 50  0001 C CNN
 F 1 "+5V" H 3315 1023 50  0000 C CNN
 F 2 "" H 3300 850 50  0001 C CNN
@@
 A13
 Wire Wire Line
-	3850 2150 3850 3000
-Wire Wire Line
-	3850 3000 2350 3000
+	4100 2150 4100 3000
+Wire Wire Line
+	4100 3000 2350 3000
 Connection ~ 2350 3000
 Wire Wire Line
 	2350 3000 2350 3100
 $Comp
-L power:GND #PWR02
+L power:GND #PWR04
 U 1 1 60C502CE
 P 1000 4500
-F 0 "#PWR02" H 1000 4250 50  0001 C CNN
+F 0 "#PWR04" H 1000 4250 50  0001 C CNN
 F 1 "GND" H 1005 4327 50  0000 C CNN
 F 2 "" H 1000 4500 50  0001 C CNN
@@
 $EndComp
 $Comp
-L power:+5V #PWR01
+L power:+5V #PWR03
 U 1 1 60C509EC
 P 1000 4200
-F 0 "#PWR01" H 1000 4050 50  0001 C CNN
+F 0 "#PWR03" H 1000 4050 50  0001 C CNN
 F 1 "+5V" H 1015 4373 50  0000 C CNN
 F 2 "" H 1000 4200 50  0001 C CNN
@@
 $EndComp
 Wire Wire Line
-	4300 2150 3850 2150
-Connection ~ 3850 2150
+	4300 2150 4100 2150
 Wire Wire Line
 	3300 1000 3750 1000
@@
 	6350 1850 6350 2050
 $Comp
-L power:GND #PWR09
+L power:GND #PWR011
 U 1 1 60CCD621
 P 6350 2050
-F 0 "#PWR09" H 6350 1800 50  0001 C CNN
+F 0 "#PWR011" H 6350 1800 50  0001 C CNN
 F 1 "GND" H 6355 1877 50  0000 C CNN
 F 2 "" H 6350 2050 50  0001 C CNN
@@
 $EndComp
 $Comp
-L power:+5V #PWR07
+L power:+5V #PWR09
 U 1 1 60CCFF23
 P 6100 3150
-F 0 "#PWR07" H 6100 3000 50  0001 C CNN
+F 0 "#PWR09" H 6100 3000 50  0001 C CNN
 F 1 "+5V" H 6115 3323 50  0000 C CNN
 F 2 "" H 6100 3150 50  0001 C CNN
@@
 $EndComp
 $Comp
-L power:GND #PWR08
+L power:GND #PWR010
 U 1 1 60CD04AE
 P 6100 3600
-F 0 "#PWR08" H 6100 3350 50  0001 C CNN
+F 0 "#PWR010" H 6100 3350 50  0001 C CNN
 F 1 "GND" H 6105 3427 50  0000 C CNN
 F 2 "" H 6100 3600 50  0001 C CNN
@@
 	5050 1850 5600 1850
 $Comp
-L power:+5V #PWR03
+L power:+5V #PWR05
 U 1 1 60D06901
 P 1250 1350
-F 0 "#PWR03" H 1250 1200 50  0001 C CNN
+F 0 "#PWR05" H 1250 1200 50  0001 C CNN
 F 1 "+5V" H 1265 1523 50  0000 C CNN
 F 2 "" H 1250 1350 50  0001 C CNN
@@
 $EndComp
 $Comp
-L power:GND #PWR04
+L power:GND #PWR06
 U 1 1 60D06F66
 P 1250 1700
-F 0 "#PWR04" H 1250 1450 50  0001 C CNN
+F 0 "#PWR06" H 1250 1450 50  0001 C CNN
 F 1 "GND" H 1255 1527 50  0000 C CNN
 F 2 "" H 1250 1700 50  0001 C CNN
@@
 	1    1250 1700
 	1    0    0    -1
-$EndComp
-$Comp
-L Connector:XLR3_Switched J1
-U 2 1 60D12038
-P 1700 1550
-F 0 "J1" H 1700 1183 50  0000 C CNN
-F 1 "XLR3_Switched" H 1700 1274 50  0000 C CNN
-F 2 "" H 1700 1650 50  0001 C CNN
-F 3 " ~" H 1700 1650 50  0001 C CNN
-	2    1700 1550
-	-1   0    0    1
 $EndComp
 Wire Wire Line
@@
 ROM_W
 NoConn ~ 4050 4500
-NoConn ~ 1700 1550
+Text Label 3250 2150 0    50   ~ 0
+Prog
+$Comp
+L power:+5V #PWR01
+U 1 1 610701B5
+P 750 2350
+F 0 "#PWR01" H 750 2200 50  0001 C CNN
+F 1 "+5V" H 765 2523 50  0000 C CNN
+F 2 "" H 750 2350 50  0001 C CNN
+F 3 "" H 750 2350 50  0001 C CNN
+	1    750  2350
+	1    0    0    -1
+$EndComp
+$Comp
+L power:GND #PWR02
+U 1 1 610701BB
+P 750 2700
+F 0 "#PWR02" H 750 2450 50  0001 C CNN
+F 1 "GND" H 755 2527 50  0000 C CNN
+F 2 "" H 750 2700 50  0001 C CNN
+F 3 "" H 750 2700 50  0001 C CNN
+	1    750  2700
+	1    0    0    -1
+$EndComp
+Wire Wire Line
+	750  2350 750  2450
+Wire Wire Line
+	750  2450 900  2450
+Wire Wire Line
+	900  2650 750  2650
+Wire Wire Line
+	750  2650 750  2700
 Wire Wire Line
 	3250 2350 5250 2350
-Wire Wire Line
-	3250 2150 3850 2150
 Wire Bus Line
 	2050 2650 2050 3400
@@
 Wire Bus Line
 	1850 4150 3650 4150
+Text Label 1500 2550 0    50   ~ 0
+Prog
+$Comp
+L Connector:XLR3_Switched J1
+U 2 1 6107A431
+P 1700 1550
+F 0 "J1" H 1700 1183 50  0000 C CNN
+F 1 "XLR3_Switched" H 1700 1274 50  0000 C CNN
+F 2 "" H 1700 1650 50  0001 C CNN
+F 3 " ~" H 1700 1650 50  0001 C CNN
+	2    1700 1550
+	-1   0    0    1
+$EndComp
+$Comp
+L Connector:XLR3_Switched J3
+U 2 1 6107B195
+P 1200 2550
+F 0 "J3" H 1200 2183 50  0000 C CNN
+F 1 "XLR3_Switched" H 1200 2274 50  0000 C CNN
+F 2 "" H 1200 2650 50  0001 C CNN
+F 3 " ~" H 1200 2650 50  0001 C CNN
+	2    1200 2550
+	-1   0    0    1
+$EndComp
 $EndSCHEMATC
