File: hard/secondVersion/cpuBoard/cpuBoard.sch (KiCad schematic (older format))
At the start: 12 parts, among them J1 myBus, SW1 SW_Push, U1 w65c816s

Commit message: Debug clock
Parts:
- added R7: 3.3k, symbol Device:R
- R4: value (Not on board) -> 3.3k
Connections:
- net +5V: now also R7.2
- net BE: now also R7.1
Other:
- moved on the sheet: R2, R3
Changed lines of the file:
@@
 U 1 1 603FA72C
 P 5650 2350
-F 0 "R6" H 5720 2396 50  0000 L CNN
-F 1 "330R" H 5720 2305 50  0000 L CNN
+F 0 "R6" V 5443 2350 50  0000 C CNN
+F 1 "330R" V 5534 2350 50  0000 C CNN
 F 2 "" V 5580 2350 50  0001 C CNN
 F 3 "~" H 5650 2350 50  0001 C CNN
@@
 L Device:R R3
 U 1 1 60405C4D
-P 2650 2250
-F 0 "R3" H 2720 2296 50  0000 L CNN
-F 1 "3.3K" H 2720 2205 50  0000 L CNN
-F 2 "" V 2580 2250 50  0001 C CNN
-F 3 "~" H 2650 2250 50  0001 C CNN
-	1    2650 2250
+P 2550 2250
+F 0 "R3" H 2620 2296 50  0000 L CNN
+F 1 "3.3K" H 2620 2205 50  0000 L CNN
+F 2 "" V 2480 2250 50  0001 C CNN
+F 3 "~" H 2550 2250 50  0001 C CNN
+	1    2550 2250
 	1    0    0    -1
 $EndComp
@@
 L Device:R R2
 U 1 1 60406704
-P 2500 2450
-F 0 "R2" H 2570 2496 50  0000 L CNN
-F 1 "3.3K" H 2570 2405 50  0000 L CNN
-F 2 "" V 2430 2450 50  0001 C CNN
-F 3 "~" H 2500 2450 50  0001 C CNN
-	1    2500 2450
+P 2300 2450
+F 0 "R2" H 2231 2496 50  0000 R CNN
+F 1 "3.3K" H 2231 2405 50  0000 R CNN
+F 2 "" V 2230 2450 50  0001 C CNN
+F 3 "~" H 2300 2450 50  0001 C CNN
+	1    2300 2450
 	1    0    0    -1
 $EndComp
@@
 $EndComp
 Wire Wire Line
-	2650 2100 2650 2000
-Wire Wire Line
-	2650 2000 2900 2000
-Wire Wire Line
-	2650 2000 2500 2000
-Wire Wire Line
-	2500 2000 2500 2300
-Connection ~ 2650 2000
-Wire Wire Line
-	2650 2400 3200 2400
-Wire Wire Line
-	2500 2600 3200 2600
+	2550 2100 2550 2000
+Wire Wire Line
+	2550 2000 2900 2000
+Wire Wire Line
+	2550 2000 2300 2000
+Wire Wire Line
+	2300 2000 2300 2300
+Connection ~ 2550 2000
+Wire Wire Line
+	2550 2400 3200 2400
+Wire Wire Line
+	2300 2600 3200 2600
 $Comp
 L Device:LED D1
@@
 U 1 1 6040F90D
 P 1550 2700
-F 0 "R1" H 1620 2746 50  0000 L CNN
-F 1 "470R" H 1620 2655 50  0000 L CNN
+F 0 "R1" V 1343 2700 50  0000 C CNN
+F 1 "470R" V 1434 2700 50  0000 C CNN
 F 2 "" V 1480 2700 50  0001 C CNN
 F 3 "~" H 1550 2700 50  0001 C CNN
@@
 U 1 1 606205FC
 P 3050 1850
-F 0 "R4" H 3120 1896 50  0000 L CNN
-F 1 "(Not on board)" H 3120 1805 50  0000 L CNN
+F 0 "R4" H 2980 1804 50  0000 R CNN
+F 1 "3.3k" H 2980 1895 50  0000 R CNN
 F 2 "" V 2980 1850 50  0001 C CNN
 F 3 "~" H 3050 1850 50  0001 C CNN
@@
 $EndComp
 Wire Wire Line
-	2500 2000 2300 2000
-Wire Wire Line
 	2300 2000 2300 1700
-Connection ~ 2500 2000
+Connection ~ 2300 2000
 Wire Wire Line
 	3050 1700 2300 1700
@@
 	1    0    0    -1
 $EndComp
-Wire Bus Line
-	2700 3000 2700 4100
-Wire Bus Line
-	4650 3700 4650 4400
-Wire Bus Line
-	4750 2900 4750 4750
-Wire Bus Line
-	2100 5000 3700 5000
-Wire Bus Line
-	3800 5150 4500 5150
 $Comp
 L 6502_comp:myBus J1
@@
 Entry Wire Line
 	3600 5100 3700 5000
+$Comp
+L Device:R R7
+U 1 1 61B1D7C7
+P 5100 2700
+F 0 "R7" V 5307 2700 50  0000 C CNN
+F 1 "3.3k" V 5216 2700 50  0000 C CNN
+F 2 "" V 5030 2700 50  0001 C CNN
+F 3 "~" H 5100 2700 50  0001 C CNN
+	1    5100 2700
+	0    -1   -1   0
+$EndComp
+Wire Wire Line
+	4250 2500 4850 2500
+Wire Wire Line
+	4850 2500 4850 2700
+Wire Wire Line
+	4850 2700 4950 2700
+$Comp
+L power:+5V #PWR010
+U 1 1 61B246AA
+P 5400 2650
+F 0 "#PWR010" H 5400 2500 50  0001 C CNN
+F 1 "+5V" H 5415 2823 50  0000 C CNN
+F 2 "" H 5400 2650 50  0001 C CNN
+F 3 "" H 5400 2650 50  0001 C CNN
+	1    5400 2650
+	1    0    0    -1
+$EndComp
+Wire Wire Line
+	5250 2700 5400 2700
+Wire Wire Line
+	5400 2700 5400 2650
+Wire Bus Line
+	4650 3700 4650 4400
+Wire Bus Line
+	3800 5150 4500 5150
+Wire Bus Line
+	4750 2900 4750 4750
+Wire Bus Line
+	2700 3000 2700 4100
+Wire Bus Line
+	2100 5000 3700 5000
 $EndSCHEMATC
