File: schematics/esp.kicad_sch (KiCad schematic)
At the start: 3 parts

Commit message: Renaming to Marcus
Connections:
- new net: U22. (VIN), U23. (LV4) (x4)
- new net: J20. (VCC), U23. (LV4) (x2)
Changed lines of the file:
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@@
 		)
 		(instances
-			(project "markus"
+			(project "marcus"
 				(path "/03a78ca6-eaff-4f05-be7b-36cd15f8b56d/e7a10e58-ebc2-481e-bdbc-3183aa203334"
 					(reference "#PWR099")
@@
 		)
 		(instances
-			(project "markus"
+			(project "marcus"
 				(path "/03a78ca6-eaff-4f05-be7b-36cd15f8b56d/e7a10e58-ebc2-481e-bdbc-3183aa203334"
 					(reference "#PWR098")
@@
 		)
 		(instances
-			(project "markus"
+			(project "marcus"
 				(path "/03a78ca6-eaff-4f05-be7b-36cd15f8b56d/e7a10e58-ebc2-481e-bdbc-3183aa203334"
 					(reference "#PWR097")

Commit message: Update schematics for latest KiCad
Connections:
- new net: U22. (3V3), U23. (HV4) (x4)
- new net: J20. (Tx), U23. (HV4) (x2)
Changed lines of the file:
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@@
 (kicad_sch
-	(version 20231120)
+	(version 20250114)
 	(generator "eeschema")
-	(generator_version "8.0")
+	(generator_version "9.0")
 	(paper "A4")
 	(junction

Commit message: Add resistor to clock in peripherals board
Parts:
- J20, U22, U23: value ~ -> (none)
Connections:
- new net: U22. (3V3), U23. (HV4) (x4)
- new net: J20. (Tx), U23. (HV4) (x2)
