File: schematics/uart.kicad_sch (KiCad schematic)
At the start: 9 parts, among them J8 myBus, U8 74HC238, U9 W65C51N, X1 CXO_DIP8

Commit message: Add resistor to clock in peripherals board
Parts:
- J27, J7: value ~ -> (none)
