File: schematics/marcus.kicad_sch (KiCad schematic)
At the start: 0 parts

Commit message: Renaming to Marcus
Other:
- title: Markus -> Marcus
Changed lines of the file:
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@@
 	(paper "A4")
 	(title_block
-		(title "Markus")
+		(title "Marcus")
 	)
 	(wire
@@
 		)
 		(instances
-			(project "markus"
+			(project "marcus"
 				(path "/03a78ca6-eaff-4f05-be7b-36cd15f8b56d"
 					(page "2")
@@
 		)
 		(instances
-			(project "markus"
+			(project "marcus"
 				(path "/03a78ca6-eaff-4f05-be7b-36cd15f8b56d"
 					(page "12")
@@
 		)
 		(instances
-			(project "markus"
+			(project "marcus"
 				(path "/03a78ca6-eaff-4f05-be7b-36cd15f8b56d"
 					(page "7")
@@
 		)
 		(instances
-			(project "markus"
+			(project "marcus"
 				(path "/03a78ca6-eaff-4f05-be7b-36cd15f8b56d"
 					(page "4")
@@
 		)
 		(instances
-			(project "markus"
+			(project "marcus"
 				(path "/03a78ca6-eaff-4f05-be7b-36cd15f8b56d"
 					(page "5")
@@
 		)
 		(instances
-			(project "markus"
+			(project "marcus"
 				(path "/03a78ca6-eaff-4f05-be7b-36cd15f8b56d"
 					(page "8")
@@
 		)
 		(instances
-			(project "markus"
+			(project "marcus"
 				(path "/03a78ca6-eaff-4f05-be7b-36cd15f8b56d"
 					(page "10")
@@
 		)
 		(instances
-			(project "markus"
+			(project "marcus"
 				(path "/03a78ca6-eaff-4f05-be7b-36cd15f8b56d"
 					(page "9")
@@
 		)
 		(instances
-			(project "markus"
+			(project "marcus"
 				(path "/03a78ca6-eaff-4f05-be7b-36cd15f8b56d"
 					(page "3")
@@
 		)
 		(instances
-			(project "markus"
+			(project "marcus"
 				(path "/03a78ca6-eaff-4f05-be7b-36cd15f8b56d"
 					(page "11")
@@
 		)
 		(instances
-			(project "markus"
+			(project "marcus"
 				(path "/03a78ca6-eaff-4f05-be7b-36cd15f8b56d"
 					(page "6")
@@
 		)
 		(instances
-			(project "markus"
+			(project "marcus"
 				(path "/03a78ca6-eaff-4f05-be7b-36cd15f8b56d"
 					(page "13")

Commit message: Update schematics for peripherals
Other:
- added sheet All peripherals (peripherals.kicad_sch)
Changed lines of the file:
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@@
+		)
+	)
+	(sheet
+		(at 57.15 162.56)
+		(size 53.34 13.97)
+		(exclude_from_sim no)
+		(in_bom yes)
+		(on_board yes)
+		(dnp no)
+		(fields_autoplaced yes)
+		(stroke
+			(width 0.1524)
+			(type solid)
+		)
+		(fill
+			(color 0 0 0 0.0000)
+		)
+		(property "Sheetname" "All peripherals"
+			(at 57.15 161.8484 0)
+			(effects
+				(font
+					(size 1.27 1.27)
+				)
+				(justify left bottom)
+			)
+		)
+		(property "Sheetfile" "peripherals.kicad_sch"
+			(at 57.15 177.1146 0)
+			(effects
+				(font
+					(size 1.27 1.27)
+				)
+				(justify left top)
+			)
+		)
+		(instances
+			(project "marcus"
+				(path "/03a78ca6-eaff-4f05-be7b-36cd15f8b56d"
+					(page "14")
+				)
+			)
 		)
 	)

Commit message: Draw reset board
Other:
- added sheet reset board (reset.kicad_sch)
Changed lines of the file:
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@@
+	)
+	(sheet
+		(at 189.23 111.76)
+		(size 63.5 11.43)
+		(exclude_from_sim no)
+		(in_bom yes)
+		(on_board yes)
+		(dnp no)
+		(fields_autoplaced yes)
+		(stroke
+			(width 0.1524)
+			(type solid)
+		)
+		(fill
+			(color 0 0 0 0)
+		)
+		(property "Sheetname" "reset board"
+			(at 189.23 111.0484 0)
+			(show_name no)
+			(do_not_autoplace no)
+			(effects
+				(font
+					(size 1.27 1.27)
+				)
+				(justify left bottom)
+			)
+		)
+		(property "Sheetfile" "reset.kicad_sch"
+			(at 189.23 123.7746 0)
+			(show_name no)
+			(do_not_autoplace no)
+			(effects
+				(font
+					(size 1.27 1.27)
+				)
+				(justify left top)
+			)
+		)
+		(instances
+			(project "marcus"
+				(path "/03a78ca6-eaff-4f05-be7b-36cd15f8b56d"
+					(page "15")
+				)
+			)
+		)
 	)
 	(sheet
